File: KeyboardPCB.kicad_pcb (KiCad board)
At the start: 2 copper layers, 0 parts

Commit message: PCB File Visualized.
Parts:
- added C1: 1u, Capacitor_SMD:C_0805_2012Metric, F.Cu at (50.0, 108.6)
- added C2: 22p, Capacitor_SMD:C_0805_2012Metric, F.Cu at (50.0, 111.6)
- added C3: 22p, Capacitor_SMD:C_0805_2012Metric, F.Cu at (50.0, 114.6)
- added C4: 0.1u, Capacitor_SMD:C_0805_2012Metric, F.Cu at (50.0, 117.6)
- added C5: 0.1u, Capacitor_SMD:C_0805_2012Metric, F.Cu at (50.0, 120.6)
- added C6: 0.1u, Capacitor_SMD:C_0805_2012Metric, F.Cu at (50.0, 123.6)
- added C7: 0.1u, Capacitor_SMD:C_0805_2012Metric, F.Cu at (50.0, 126.6)
- added C8: 0.1u, Diode_SMD:D_SOD-123, F.Cu at (70.5, 129.9)
- added D1: PRTR5V0U2X, Diode_SMD:D_SOD-123, F.Cu at (70.5, 133.2)
- added D10: D, Diode_SMD:D_SOD-123, F.Cu at (108.4, 64.8)
- added D11: D, Diode_SMD:D_SOD-123, F.Cu at (108.4, 68.2)
- added D12: D, Diode_SMD:D_SOD-123, F.Cu at (108.4, 71.5)
- added D13: D, Diode_SMD:D_SOD-123, F.Cu at (108.4, 74.9)
- added D14: D, Diode_SMD:D_SOD-123, F.Cu at (114.2, 38.0)
- added D15: D, Diode_SMD:D_SOD-123, F.Cu at (114.2, 41.4)
- added D16: D, Diode_SMD:D_SOD-123, F.Cu at (114.2, 44.7)
- added D17: D, Diode_SMD:D_SOD-123, F.Cu at (114.2, 48.1)
- added D18: D, Diode_SMD:D_SOD-123, F.Cu at (114.2, 51.4)
- added D19: D, Diode_SMD:D_SOD-123, F.Cu at (114.2, 54.8)
- added D2: D, Diode_SMD:D_SOD-123, F.Cu at (108.4, 38.0)
- added D20: D, Diode_SMD:D_SOD-123, F.Cu at (114.2, 58.1)
- added D21: D, Diode_SMD:D_SOD-123, F.Cu at (114.2, 61.5)
- added D22: D, Diode_SMD:D_SOD-123, F.Cu at (114.2, 64.8)
- added D23: D, Diode_SMD:D_SOD-123, F.Cu at (114.2, 68.2)
- added D24: D, Diode_SMD:D_SOD-123, F.Cu at (114.2, 71.5)
- added D25: D, Diode_SMD:D_SOD-123, F.Cu at (114.2, 74.9)
- added D26: D, Diode_SMD:D_SOD-123, F.Cu at (120.0, 38.0)
- added D27: D, Diode_SMD:D_SOD-123, F.Cu at (120.0, 41.4)
- added D28: D, Diode_SMD:D_SOD-123, F.Cu at (120.0, 44.7)
- added D29: D, Diode_SMD:D_SOD-123, F.Cu at (120.0, 48.1)
- added D3: D, Diode_SMD:D_SOD-123, F.Cu at (108.4, 41.4)
- added D30: D, Diode_SMD:D_SOD-123, F.Cu at (120.0, 51.4)
- added D31: D, Diode_SMD:D_SOD-123, F.Cu at (120.0, 54.8)
- added D32: D, Diode_SMD:D_SOD-123, F.Cu at (120.0, 58.1)
- added D33: D, Diode_SMD:D_SOD-123, F.Cu at (120.0, 61.5)
- added D34: D, Diode_SMD:D_SOD-123, F.Cu at (120.0, 64.8)
- added D35: D, Diode_SMD:D_SOD-123, F.Cu at (120.0, 68.2)
- added D36: D, Diode_SMD:D_SOD-123, F.Cu at (120.0, 71.5)
- added D37: D, Diode_SMD:D_SOD-123, F.Cu at (120.0, 74.9)
- added D38: D, Diode_SMD:D_SOD-123, F.Cu at (125.8, 38.0)
- added D39: D, Diode_SMD:D_SOD-123, F.Cu at (125.8, 41.4)
- added D4: D, Diode_SMD:D_SOD-123, F.Cu at (108.4, 44.7)
- added D40: D, Diode_SMD:D_SOD-123, F.Cu at (125.8, 44.7)
- added D41: D, Diode_SMD:D_SOD-123, F.Cu at (125.8, 48.1)
- added D42: D, Diode_SMD:D_SOD-123, F.Cu at (125.8, 51.4)
- added D43: D, Diode_SMD:D_SOD-123, F.Cu at (125.8, 54.8)
- added D44: D, Diode_SMD:D_SOD-123, F.Cu at (125.8, 58.1)
- added D45: D, Diode_SMD:D_SOD-123, F.Cu at (125.8, 61.5)
- added D46: D, Diode_SMD:D_SOD-123, F.Cu at (125.8, 64.8)
- added D47: D, Diode_SMD:D_SOD-123, F.Cu at (125.8, 68.2)
- added D48: D, Diode_SMD:D_SOD-123, F.Cu at (125.8, 71.5)
- added D49: D, Diode_SMD:D_SOD-123, F.Cu at (125.8, 74.9)
- added D5: D, Diode_SMD:D_SOD-123, F.Cu at (108.4, 48.1)
- added D50: D, Diode_SMD:D_SOD-123, F.Cu at (131.6, 38.0)
- added D51: D, Diode_SMD:D_SOD-123, F.Cu at (131.6, 41.4)
- added D52: D, Diode_SMD:D_SOD-123, F.Cu at (131.6, 44.7)
- added D53: D, Diode_SMD:D_SOD-123, F.Cu at (131.6, 48.1)
- added D54: D, Diode_SMD:D_SOD-123, F.Cu at (131.6, 51.4)
- added D55: D, Diode_SMD:D_SOD-123, F.Cu at (131.6, 54.8)
- added D56: D, Diode_SMD:D_SOD-123, F.Cu at (131.6, 58.1)
- added D57: D, Diode_SMD:D_SOD-123, F.Cu at (131.6, 61.5)
- added D58: D, Diode_SMD:D_SOD-123, F.Cu at (131.6, 64.8)
- added D59: D, Diode_SMD:D_SOD-123, F.Cu at (131.6, 68.2)
- added D6: D, Diode_SMD:D_SOD-123, F.Cu at (108.4, 51.4)
- added D60: D, Diode_SMD:D_SOD-123, F.Cu at (131.6, 71.5)
- added D61: D, Diode_SMD:D_SOD-123, F.Cu at (131.6, 74.9)
- added D62: D, Diode_SMD:D_SOD-123, F.Cu at (137.4, 38.0)
- added D63: D, Diode_SMD:D_SOD-123, F.Cu at (137.4, 41.4)
- added D64: D, Diode_SMD:D_SOD-123, F.Cu at (137.4, 44.7)
- added D65: D, Diode_SMD:D_SOD-123, F.Cu at (137.4, 48.1)
- added D66: D, Diode_SMD:D_SOD-123, F.Cu at (137.4, 51.4)
- added D67: D, Diode_SMD:D_SOD-123, F.Cu at (137.4, 54.8)
- added D68: D, Diode_SMD:D_SOD-123, F.Cu at (137.4, 58.1)
- added D7: D, Diode_SMD:D_SOD-123, F.Cu at (108.4, 54.8)
- added D8: D, Diode_SMD:D_SOD-123, F.Cu at (108.4, 58.1)
- added D9: D, Diode_SMD:D_SOD-123, F.Cu at (108.4, 61.5)
- added F1: 500m, Fuse:Fuse_1206_3216Metric_Pad1.42x1.75mm_HandSolder, F.Cu at (59.9, 133.8)
- added J1: AVR-ISP-6, random-keyboard-parts:D_SOD-123-Pretty, F.Cu at (74.2, 108.8)
- added R1: 10k, Resistor_SMD:R_0805_2012Metric_Pad1.20x1.40mm_HandSolder, F.Cu at (54.6, 108.6)
- added R2: 10k, Resistor_SMD:R_0805_2012Metric_Pad1.20x1.40mm_HandSolder, F.Cu at (54.6, 111.5)
- added R3: 22, Resistor_SMD:R_0805_2012Metric_Pad1.20x1.40mm_HandSolder, F.Cu at (54.6, 114.5)
- added R4: 22, Resistor_SMD:R_0805_2012Metric_Pad1.20x1.40mm_HandSolder, F.Cu at (54.6, 117.4)
- added R5: 5.1k, Resistor_SMD:R_0805_2012Metric_Pad1.20x1.40mm_HandSolder, F.Cu at (54.6, 120.4)
- added R6: 5.1k, Resistor_SMD:R_0805_2012Metric_Pad1.20x1.40mm_HandSolder, F.Cu at (54.6, 123.3)
- added SW1: GRV, Alps_Only:ALPS-1U, F.Cu at (51.9, 42.5)
- added SW10: #9, Alps_Only:ALPS-1U, F.Cu at (51.9, 104.3)
- added SW11: #0, Alps_Only:ALPS-1U, F.Cu at (60.1, 42.5)
- added SW12: -_, Alps_Only:ALPS-1U, F.Cu at (60.1, 49.3)
- added SW13: =+, Alps_Only:ALPS-1U, F.Cu at (60.1, 56.2)
- added SW14: BSPC, Alps_Only:ALPS-2U, F.Cu at (60.1, 63.1)
- added SW15: PGUP, Alps_Only:ALPS-1U, F.Cu at (60.1, 70.0)
- added SW16: TAB, Alps_Only:ALPS-1.5U, F.Cu at (60.1, 76.8)
- added SW17: Q, Alps_Only:ALPS-1U, F.Cu at (60.1, 83.7)
- added SW18: W, Alps_Only:ALPS-1U, F.Cu at (60.1, 90.6)
- added SW19: E, Alps_Only:ALPS-1U, F.Cu at (60.1, 97.5)
- added SW2: #1, Alps_Only:ALPS-1U, F.Cu at (51.9, 49.3)
- added SW20: R, Alps_Only:ALPS-1U, F.Cu at (60.1, 104.3)
- added SW21: T, Alps_Only:ALPS-1U, F.Cu at (68.4, 42.5)
- added SW22: Y, Alps_Only:ALPS-1U, F.Cu at (68.4, 49.3)
- added SW23: U, Alps_Only:ALPS-1U, F.Cu at (68.4, 56.2)
- added SW24: I, Alps_Only:ALPS-1U, F.Cu at (68.4, 63.1)
- added SW25: O, Alps_Only:ALPS-1U, F.Cu at (68.4, 70.0)
- added SW26: P, Alps_Only:ALPS-1U, F.Cu at (68.4, 76.8)
- added SW27: [{, Alps_Only:ALPS-1U, F.Cu at (68.4, 83.7)
- added SW28: ]}, Alps_Only:ALPS-1U, F.Cu at (68.4, 90.6)
- added SW29: \|, Alps_Only:ALPS-1.5U, F.Cu at (68.4, 97.5)
- added SW3: #2, Alps_Only:ALPS-1U, F.Cu at (51.9, 56.2)
- added SW30: PGDN, Alps_Only:ALPS-1U, F.Cu at (68.4, 104.3)
- added SW31: CAPSLOCK, Alps_Only:ALPS-1.75U, F.Cu at (76.6, 42.5)
- added SW32: A, Alps_Only:ALPS-1U, F.Cu at (76.6, 49.3)
- added SW33: S, Alps_Only:ALPS-1U, F.Cu at (76.6, 56.2)
- added SW34: D, Alps_Only:ALPS-1U, F.Cu at (76.6, 63.1)
- added SW35: F, Alps_Only:ALPS-1U, F.Cu at (76.6, 70.0)
- added SW36: G, Alps_Only:ALPS-1U, F.Cu at (76.6, 76.8)
- added SW37: H, Alps_Only:ALPS-1U, F.Cu at (76.6, 83.7)
- added SW38: J, Alps_Only:ALPS-1U, F.Cu at (76.6, 90.6)
- added SW39: K, Alps_Only:ALPS-1U, F.Cu at (76.6, 97.5)
- added SW4: #3, Alps_Only:ALPS-1U, F.Cu at (51.9, 63.1)
- added SW40: L, Alps_Only:ALPS-1U, F.Cu at (76.6, 104.3)
- added SW41: ;:, Alps_Only:ALPS-1U, F.Cu at (84.9, 42.5)
- added SW42: '", Alps_Only:ALPS-1U, F.Cu at (84.9, 49.3)
- added SW43: ENTER, Alps_Only:ALPS-2.25U, F.Cu at (84.9, 56.2)
- added SW44: INS, Alps_Only:ALPS-1U, F.Cu at (84.9, 63.1)
- added SW45: LSHIFT, Alps_Only:ALPS-2.25U, F.Cu at (84.9, 70.0)
- added SW46: Z, Alps_Only:ALPS-1U, F.Cu at (84.9, 76.8)
- added SW47: X, Alps_Only:ALPS-1U, F.Cu at (84.9, 83.7)
- added SW48: C, Alps_Only:ALPS-1U, F.Cu at (84.9, 90.6)
- added SW49: V, Alps_Only:ALPS-1U, F.Cu at (84.9, 97.5)
- added SW5: #4, Alps_Only:ALPS-1U, F.Cu at (51.9, 70.0)
- added SW50: B, Alps_Only:ALPS-1U, F.Cu at (84.9, 104.3)
- added SW51: N, Alps_Only:ALPS-1U, F.Cu at (93.1, 42.5)
- added SW52: M, Alps_Only:ALPS-1U, F.Cu at (93.1, 49.3)
- added SW53: ,<, Alps_Only:ALPS-1U, F.Cu at (93.1, 56.2)
- added SW54: .>, Alps_Only:ALPS-1U, F.Cu at (93.1, 63.1)
- added SW55: /?, Alps_Only:ALPS-1U, F.Cu at (93.1, 70.0)
- added SW56: RSHIFT, Alps_Only:ALPS-1.75U, F.Cu at (93.1, 76.8)
- added SW57: UP, Alps_Only:ALPS-1U, F.Cu at (93.1, 83.7)
- added SW58: DEL, Alps_Only:ALPS-1U, F.Cu at (93.1, 90.6)
- added SW59: LCTRL, Alps_Only:ALPS-1.5U, F.Cu at (93.1, 97.5)
- added SW6: #5, Alps_Only:ALPS-1U, F.Cu at (51.9, 76.8)
- added SW60: LALT, Alps_Only:ALPS-1.25U, F.Cu at (93.1, 104.3)
- added SW61: LCMD, Alps_Only:ALPS-1.5U, F.Cu at (101.4, 42.5)
- added SW62: SPACE, Alps_Only:ALPS-6.5U, F.Cu at (101.4, 49.3)
- added SW63: RCOMMAND, Alps_Only:ALPS-1U, F.Cu at (101.4, 56.2)
- added SW64: RALT, Alps_Only:ALPS-1.25U, F.Cu at (101.4, 63.1)
- added SW65: LEFT, Alps_Only:ALPS-1U, F.Cu at (101.4, 70.0)
- added SW66: DOWN, Alps_Only:ALPS-1U, F.Cu at (101.4, 76.8)
- added SW67: RIGHT, Alps_Only:ALPS-1U, F.Cu at (101.4, 83.7)
- added SW68: SW_SKQG, Button_Switch_SMD:SW_SPST_SKQG_WithStem, F.Cu at (72.4, 124.8)
- added SW7: #6, Alps_Only:ALPS-1U, F.Cu at (51.9, 83.7)
- added SW8: #7, Alps_Only:ALPS-1U, F.Cu at (51.9, 90.6)
- added SW9: #8, Alps_Only:ALPS-1U, F.Cu at (51.9, 97.5)
- added U1: ATmega32U4-A, Package_QFP:TQFP-44_10x10mm_P0.8mm, F.Cu at (64.1, 114.3)
- added USB1: HRO-TYPE-C-31-M-12, Type-C:HRO-TYPE-C-31-M-12-HandSoldering, F.Cu at (62.3, 131.3)
- added Y1: Crystal_GND24_Small, Crystal:Crystal_SMD_3225-4Pin_3.2x2.5mm, F.Cu at (73.9, 112.7)
