File: KeyboardPCB.kicad_pcb (KiCad board)
At the start: 2 copper layers, 155 parts, among them J1 AVR-ISP-6, SW1 GRV, SW10 #9, SW11 #0, SW12 -_, SW13 =+, SW14 BSPC, SW15 PGUP, SW16 TAB, SW17 Q, SW18 W, SW19 E, SW2 #1, SW20 R, SW21 T, SW22 Y, SW23 U, SW24 I, SW25 O, SW26 P, SW27 [{, SW28 ]}, SW29 \|, SW3 #2, SW30 PGDN, SW31 CAPSLOCK, SW32 A, SW33 S, SW34 D, SW35 F, SW36 G, SW37 H, SW38 J, SW39 K, SW4 #3, SW40 L, SW41 ;:, SW42 '", SW43 ENTER, SW44 INS, SW45 LSHIFT, SW46 Z, SW47 X, SW48 C, SW49 V, SW5 #4, SW50 B, SW51 N, SW52 M, SW53 ,<, SW54 .>, SW55 /?, SW56 RSHIFT, SW57 UP, SW58 DEL, SW59 LCTRL, SW6 #5, SW60 LALT, SW61 LCMD, SW62 SPACE, SW63 RCOMMAND, SW64 RALT, SW65 LEFT, SW66 DOWN, SW67 RIGHT, SW68 SW_SKQG, SW7 #6, SW8 #7, SW9 #8, U1 ATmega32U4-A, Y1 Crystal_GND24_Small

Commit message: Keyboard keys positioned
Parts:
- C1, C2, C3, C4, C5, C6, C7, C8, D10, D11, D12, D13, D14, D15, D16, D17, D18, D19, D2, D20, D21, D22, D23, D24, D25, D26, D27, D28, D29, D3, D30, D31, D32, D33, D34, D35, D36, D37, D38, D39, D4, D40, D41, D42, D43, D44, D45, D46, D47, D48, D49, D5, D50, D51, D52, D53, D54, D55, D56, D57, D58, D59, D6, D60, D61, D62, D63, D64, D65, D66, D67, D68, D7, D8, D9, F1, R1, R2, R3, R4, R5, R6, SW68, U1, USB1, Y1: moved to B.Cu
- D1: footprint Diode_SMD:D_SOD-123 -> random-keyboard-parts:SOT143B; moved to B.Cu
- J1: footprint random-keyboard-parts:D_SOD-123-Pretty -> random-keyboard-parts:Reset_Pretty-Mask; moved to B.Cu
- SW61: value LCMD -> LCOMMAND
- moved SW15 324.4 mm to (381.7, 26.7)
- moved SW30 318.7 mm to (381.7, 45.8)
- moved SW44 296.8 mm to (381.7, 64.8)
- moved SW14 295.2 mm to (353.1, 26.7)
- moved SW29 294.0 mm to (357.8, 45.8)
- moved SW58 288.4 mm to (381.5, 83.8)
- moved SW67 280.8 mm to (381.5, 102.9)
- moved SW28 269.4 mm to (334.0, 45.8)
- moved SW57 269.3 mm to (362.5, 83.8)
- moved SW13 266.0 mm to (324.5, 26.8)
- moved SW43 266.0 mm to (350.7, 64.8)
- moved SW66 262.4 mm to (362.5, 102.9)
- moved SW27 249.5 mm to (315.0, 45.8)
- moved SW12 246.4 mm to (305.5, 26.8)
- moved SW65 244.3 mm to (343.4, 102.9)
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
Commit message: Layout progress.
Moved the diodes to each of their keys.
Mostly finished placing capacitors, resistors, and other components.
Parts:
- moved D67 286.6 mm to (351.5, 160.4), turned to 90 degrees
- moved D58 279.9 mm to (351.5, 141.2), turned to 90 degrees
- moved D44 274.6 mm to (351.5, 122.2), turned to 90 degrees
- moved D30 270.0 mm to (351.5, 103.2), turned to 90 degrees
- moved D66 267.9 mm to (332.4, 160.4), turned to 90 degrees
- moved D15 265.4 mm to (351.5, 84.1), turned to 90 degrees
- moved D57 260.8 mm to (332.4, 141.2), turned to 90 degrees
- moved D65 249.3 mm to (313.4, 160.3), turned to 90 degrees
- moved D29 245.9 mm to (327.7, 103.2), turned to 90 degrees
- moved D43 243.5 mm to (320.5, 122.3), turned to 90 degrees
- moved D14 236.7 mm to (322.9, 84.1), turned to 90 degrees
- moved D56 234.6 mm to (306.3, 141.3), turned to 90 degrees
- moved D64 228.5 mm to (292.0, 160.4), turned to 90 degrees
- moved D28 221.9 mm to (303.9, 103.2), turned to 90 degrees
- moved Y1 221.2 mm to (244.0, 161.2)
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- renumbered D1 to D0, D2 to D1, D11 to D10, D12 to D11, D13 to D12, D14 to D13, D15 to D14, D16 to D15, D17 to D16, D18 to D17, D19 to D18, D20 to D19, D3 to D2, D21 to D20, D22 to D21, D23 to D22, D24 to D23, D25 to D24, D26 to D25, D27 to D26, D28 to D27, D29 to D28, D30 to D29, D4 to D3, D31 to D30, D32 to D31, D33 to D32, D34 to D33, D35 to D34, D36 to D35, D37 to D36, D38 to D37, D39 to D38, D40 to D39, D5 to D4, D41 to D40, D42 to D41, D43 to D42, D44 to D43, D45 to D44, D46 to D45, D47 to D46, D48 to D47, D49 to D48, D50 to D49, D6 to D5, D51 to D50, D52 to D51, D53 to D52, D54 to D53, D55 to D54, D56 to D55, D57 to D56, D58 to D57, D59 to D58, D60 to D59, D7 to D6, D61 to D60, D62 to D61, D63 to D62, D64 to D63, D65 to D64, D66 to D65, D67 to D66, D68 to D67, D8 to D7, D9 to D8, D10 to D9

Commit message: PCB Layout finished.
Placed all components on the board.
Figured out where all the decoupling capacitors go!
Also fixed an issue with one of the decoupling capacitors not being 10 uF.
Parts:
- C8: value 0.1u -> 10u; footprint Diode_SMD:D_SOD-123 -> Capacitor_SMD:C_0805_2012Metric
- moved F1 92.7 mm to (200.3, 85.1), turned to 90 degrees
- moved SW68 72.5 mm to (249.5, 157.4), turned to 90 degrees
- moved C8 48.1 mm to (214.7, 147.1)
- moved C7 46.0 mm to (229.6, 153.6), turned to -90 degrees
- moved C6 40.5 mm to (223.9, 147.1), turned to 180 degrees
- moved R4 31.7 mm to (219.3, 142.6), turned to 90 degrees
- moved C1 30.6 mm to (219.2, 147.1)
- moved R2 27.1 mm to (247.9, 150.3)
- moved C4 24.9 mm to (223.9, 163.8), turned to 0 degrees
- moved C5 19.1 mm to (210.6, 160.0)
- moved R3 13.0 mm to (216.9, 142.6), turned to -90 degrees
- moved C3 11.9 mm to (236.4, 159.5)
- moved C2 11.9 mm to (236.4, 157.5)
- moved Y1 11.8 mm to (232.5, 158.3)
- moved D12 9.37 mm to (266.0, 82.8)
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Other:
- board outline added: 304.8 x 100 mm
